Commit message: two cameras

File: src/capra_2dnav/models/capra6/capra6.urdf (robot description, URDF)
Before this commit: robot capra6, 5 links, 4 joints
Links:
- removed link camera
- added link camera_left, mass 1; collision sphere radius=0.1
- added link camera_right, mass 1; collision sphere radius=0.1
Joints:
- added joint joint3: type fixed, parent base_link, child camera_right, origin xyz=0.28 0.2 1.28 rpy=0 0.9 0
- joint joint2: child camera -> camera_left; origin xyz=0.28 0 1.28 rpy=0 0.92 0 -> xyz=0.28 -0.2 1.28 rpy=0 0.9 0
